File: CMPE-310-Project-5.kicad_pcb (KiCad board)
At the start: 4 copper layers, 7 parts, among them J1 DSUB-9, U1 max235cpg, U3 pkd8279, U4 8086_Min_Mode

Commit message: PCB Changes
Connections:
- U4 pad 10: unconnected-(U4-Pad10) -> /A6
- U4 pad 11: unconnected-(U4-Pad11) -> /A5
- U4 pad 12: unconnected-(U4-Pad12) -> /A4
- U4 pad 13: unconnected-(U4-Pad13) -> /A3
- U4 pad 14: unconnected-(U4-Pad14) -> /A2
- U4 pad 15: unconnected-(U4-Pad15) -> /A1
- U4 pad 2: unconnected-(U4-Pad2) -> /A14
- U4 pad 3: unconnected-(U4-Pad3) -> /A13
- U4 pad 37: unconnected-(U4-Pad37) -> /A17
- U4 pad 38: unconnected-(U4-Pad38) -> /A16
- U4 pad 39: unconnected-(U4-Pad39) -> /A15
- U4 pad 4: unconnected-(U4-Pad4) -> /A12
- U4 pad 5: unconnected-(U4-Pad5) -> /A11
- U4 pad 6: unconnected-(U4-Pad6) -> /A10
- U4 pad 7: unconnected-(U4-Pad7) -> /A9
- U4 pad 8: unconnected-(U4-Pad8) -> /A8
- U4 pad 9: unconnected-(U4-Pad9) -> /A7
