File: 28F010_sch.kicad_sch (KiCad schematic)
At the start: 13 parts

Commit message: PCB wiring
Parts:
- Bank0, Bank1: value (none) -> 28F010; footprint (none) -> parts:28F010
- U10: value (none) -> 74LVC1G332; footprint (none) -> Package_TO_SOT_SMD:SOT-23-6
- U11, U8: value (none) -> 74LS138; footprint (none) -> Package_DIP:DIP-16_W7.62mm
- U12, U15, U17, U9: value (none) -> CY7C199; footprint (none) -> Package_DIP:DIP-28_W7.62mm
- U16, U40: value (none) -> 4012; footprint (none) -> Package_DIP:DIP-12_W7.62mm
- U3, U39: value (none) -> 74LS04; footprint (none) -> Package_DIP:DIP-14_W7.62mm
Changed lines of the file:
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@@
       (effects (font (size 1.27 1.27)) (justify left))
     )
-    (property "Value" "" (id 1) (at 90.17 31.7499 90)
-      (effects (font (size 1.27 1.27)) (justify left))
-    )
-    (property "Footprint" "" (id 2) (at 85.09 30.48 0)
+    (property "Value" "74LS04" (id 1) (at 90.17 31.7499 90)
+      (effects (font (size 1.27 1.27)) (justify left))
+    )
+    (property "Footprint" "Package_DIP:DIP-14_W7.62mm" (id 2) (at 85.09 30.48 0)
       (effects (font (size 1.27 1.27)) hide)
     )
@@
       (effects (font (size 1.524 1.524)))
     )
-    (property "Value" "" (id 1) (at 210.82 86.36 0)
+    (property "Value" "28F010" (id 1) (at 210.82 86.36 0)
       (effects (font (size 1.524 1.524)))
     )
-    (property "Footprint" "" (id 2) (at 210.82 87.884 0)
+    (property "Footprint" "parts:28F010" (id 2) (at 210.82 87.884 0)
       (effects (font (size 1.524 1.524)) hide)
     )
@@
       (effects (font (size 1.27 1.27)) (justify left))
     )
-    (property "Value" "" (id 1) (at 27.94 25.3999 0)
-      (effects (font (size 1.27 1.27)) (justify left))
-    )
-    (property "Footprint" "" (id 2) (at 21.59 24.13 0)
+    (property "Value" "74LS04" (id 1) (at 27.94 25.3999 0)
+      (effects (font (size 1.27 1.27)) (justify left))
+    )
+    (property "Footprint" "Package_DIP:DIP-14_W7.62mm" (id 2) (at 21.59 24.13 0)
       (effects (font (size 1.27 1.27)) hide)
     )
@@
       (effects (font (size 1.27 1.27)) (justify left))
     )
-    (property "Value" "" (id 1) (at 74.4094 69.85 0)
-      (effects (font (size 1.27 1.27)) (justify left))
-    )
-    (property "Footprint" "" (id 2) (at 72.39 82.55 0)
+    (property "Value" "74LS138" (id 1) (at 74.4094 69.85 0)
+      (effects (font (size 1.27 1.27)) (justify left))
+    )
+    (property "Footprint" "Package_DIP:DIP-16_W7.62mm" (id 2) (at 72.39 82.55 0)
       (effects (font (size 1.27 1.27)) hide)
     )
@@
       (effects (font (size 1.27 1.27)) (justify left))
     )
-    (property "Value" "" (id 1) (at 112.5094 132.08 0)
-      (effects (font (size 1.27 1.27)) (justify left))
-    )
-    (property "Footprint" "" (id 2) (at 110.49 161.29 0)
+    (property "Value" "CY7C199" (id 1) (at 112.5094 132.08 0)
+      (effects (font (size 1.27 1.27)) (justify left))
+    )
+    (property "Footprint" "Package_DIP:DIP-28_W7.62mm" (id 2) (at 110.49 161.29 0)
       (effects (font (size 1.27 1.27)) hide)
     )
@@
       (effects (font (size 1.27 1.27)) (justify left))
     )
-    (property "Value" "" (id 1) (at 36.3094 69.85 0)
-      (effects (font (size 1.27 1.27)) (justify left))
-    )
-    (property "Footprint" "" (id 2) (at 34.29 82.55 0)
+    (property "Value" "74LS138" (id 1) (at 36.3094 69.85 0)
+      (effects (font (size 1.27 1.27)) (justify left))
+    )
+    (property "Footprint" "Package_DIP:DIP-16_W7.62mm" (id 2) (at 34.29 82.55 0)
       (effects (font (size 1.27 1.27)) hide)
     )
@@
     (in_bom yes) (on_board yes) (fields_autoplaced)
     (property "Reference" "U16" (id 0) (at 111.76 8.89 0))
-    (property "Value" "" (id 1) (at 111.76 11.43 0))
-    (property "Footprint" "" (id 2) (at 111.76 19.05 0)
+    (property "Value" "4012" (id 1) (at 111.76 11.43 0))
+    (property "Footprint" "Package_DIP:DIP-12_W7.62mm" (id 2) (at 111.76 19.05 0)
       (effects (font (size 1.27 1.27)) hide)
     )
@@
       (effects (font (size 1.27 1.27)) (justify left))
     )
-    (property "Value" "" (id 1) (at 100.33 34.2899 90)
-      (effects (font (size 1.27 1.27)) (justify left))
-    )
-    (property "Footprint" "" (id 2) (at 95.25 33.02 0)
+    (property "Value" "74LS04" (id 1) (at 100.33 34.2899 90)
+      (effects (font (size 1.27 1.27)) (justify left))
+    )
+    (property "Footprint" "Package_DIP:DIP-14_W7.62mm" (id 2) (at 95.25 33.02 0)
       (effects (font (size 1.27 1.27)) hide)
     )
@@
       (effects (font (size 1.27 1.27)) (justify left))
     )
-    (property "Value" "" (id 1) (at 36.3094 130.81 0)
-      (effects (font (size 1.27 1.27)) (justify left))
-    )
-    (property "Footprint" "" (id 2) (at 34.29 160.02 0)
+    (property "Value" "CY7C199" (id 1) (at 36.3094 130.81 0)
+      (effects (font (size 1.27 1.27)) (justify left))
+    )
+    (property "Footprint" "Package_DIP:DIP-28_W7.62mm" (id 2) (at 34.29 160.02 0)
       (effects (font (size 1.27 1.27)) hide)
     )
@@
       (effects (font (size 1.27 1.27)) (justify left))
     )
-    (property "Value" "" (id 1) (at 54.61 53.0224 90)
-      (effects (font (size 1.27 1.27)) (justify left))
-    )
-    (property "Footprint" "" (id 2) (at 49.53 52.07 0)
+    (property "Value" "74LVC1G332" (id 1) (at 54.61 53.0224 90)
+      (effects (font (size 1.27 1.27)) (justify left))
+    )
+    (property "Footprint" "Package_TO_SOT_SMD:SOT-23-6" (id 2) (at 49.53 52.07 0)
       (effects (font (size 1.27 1.27)) hide)
     )
@@
       (effects (font (size 1.27 1.27)) (justify left))
     )
-    (property "Value" "" (id 1) (at 150.6094 132.08 0)
-      (effects (font (size 1.27 1.27)) (justify left))
-    )
-    (property "Footprint" "" (id 2) (at 148.59 161.29 0)
+    (property "Value" "CY7C199" (id 1) (at 150.6094 132.08 0)
+      (effects (font (size 1.27 1.27)) (justify left))
+    )
+    (property "Footprint" "Package_DIP:DIP-28_W7.62mm" (id 2) (at 148.59 161.29 0)
       (effects (font (size 1.27 1.27)) hide)
     )
@@
       (effects (font (size 1.524 1.524)))
     )
-    (property "Value" "" (id 1) (at 209.55 22.86 0)
+    (property "Value" "28F010" (id 1) (at 209.55 22.86 0)
       (effects (font (size 1.524 1.524)))
     )
-    (property "Footprint" "" (id 2) (at 209.55 24.384 0)
+    (property "Footprint" "parts:28F010" (id 2) (at 209.55 24.384 0)
       (effects (font (size 1.524 1.524)) hide)
     )
@@
     (in_bom yes) (on_board yes) (fields_autoplaced)
     (property "Reference" "U16" (id 0) (at 111.76 19.05 0))
-    (property "Value" "" (id 1) (at 111.76 21.59 0))
-    (property "Footprint" "" (id 2) (at 111.76 29.21 0)
+    (property "Value" "4012" (id 1) (at 111.76 21.59 0))
+    (property "Footprint" "Package_DIP:DIP-12_W7.62mm" (id 2) (at 111.76 29.21 0)
       (effects (font (size 1.27 1.27)) hide)
     )
@@
       (effects (font (size 1.27 1.27)) (justify left))
     )
-    (property "Value" "" (id 1) (at 46.99 25.3999 0)
-      (effects (font (size 1.27 1.27)) (justify left))
-    )
-    (property "Footprint" "" (id 2) (at 40.64 24.13 0)
+    (property "Value" "4012" (id 1) (at 46.99 25.3999 0)
+      (effects (font (size 1.27 1.27)) (justify left))
+    )
+    (property "Footprint" "Package_DIP:DIP-12_W7.62mm" (id 2) (at 40.64 24.13 0)
       (effects (font (size 1.27 1.27)) hide)
     )
@@
       (effects (font (size 1.27 1.27)) (justify left))
     )
-    (property "Value" "" (id 1) (at 74.4094 132.08 0)
-      (effects (font (size 1.27 1.27)) (justify left))
-    )
-    (property "Footprint" "" (id 2) (at 72.39 161.29 0)
-      (effects (font (size 1.27 1.27)) hide)
-    )
+    (property "Value" "CY7C199" (id 1) (at 74.4094 132.08 0)
+      (effects (font (size 1.27 1.27)) (justify left))
+    )
+    (property "Footprint" "Package_DIP:DIP-28_W7.62mm" (id 2) (at 72.39 161.29 0)
+      (effects (font (size 1.27 1.27)) hide)
+    )
