File: Bus_sch.kicad_sch (KiCad schematic)
At the start: 9 parts, among them J15 Conn_01x03_Male, J16 Conn_01x20_Male, J17 Conn_01x16_Male, U23 74LS244, U24 74LS373, U25 74LS373, U26 74LS373, U27 74LS245, U28 74LS245

Commit message: More PCB wiring
Wired all components to eachother, did not interface everything with the 8086
Parts:
- J16: footprint (none) -> Connector_Harwin:Harwin_M20-89020xx_1x20_P2.54mm_Horizontal
- J17: footprint (none) -> Connector_Harwin:Harwin_M20-89016xx_1x16_P2.54mm_Horizontal
Changed lines of the file:
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@@
       (effects (font (size 1.27 1.27)) (justify right))
     )
-    (property "Footprint" "" (id 2) (at 278.13 128.27 0)
+    (property "Footprint" "Connector_Harwin:Harwin_M20-89016xx_1x16_P2.54mm_Horizontal" (id 2) (at 278.13 128.27 0)
       (effects (font (size 1.27 1.27)) hide)
     )
@@
       (effects (font (size 1.27 1.27)) (justify right))
     )
-    (property "Footprint" "" (id 2) (at 231.14 128.27 0)
+    (property "Footprint" "Connector_Harwin:Harwin_M20-89020xx_1x20_P2.54mm_Horizontal" (id 2) (at 231.14 128.27 0)
       (effects (font (size 1.27 1.27)) hide)
     )
