File: INTR_sch.kicad_sch (KiCad schematic)
At the start: 14 parts, among them J10 Conn_01x04_Male, J11 Conn_01x03_Male, J12 Conn_01x03_Male, J13 Conn_01x02_Male, SW2 SW_Push, U13 PAL16L8, U14 16550, U18 8259A, U19 PAL16L8, U20 pkd8279, U21 8254

Commit message: More PCB wiring
Wired all components to eachother, did not interface everything with the 8086
Parts:
- J10, J11, J12, J13: footprint Connector_Harwin:Harwin_M20-89008xx_1x08_P2.54mm_Horizontal -> (none)
Changed lines of the file:
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@@
       (effects (font (size 1.27 1.27)) (justify right))
     )
-    (property "Footprint" "Connector_Harwin:Harwin_M20-89008xx_1x08_P2.54mm_Horizontal" (id 2) (at 283.21 52.07 0)
+    (property "Footprint" "" (id 2) (at 283.21 52.07 0)
       (effects (font (size 1.27 1.27)) hide)
     )
@@
       (effects (font (size 1.27 1.27)) (justify right))
     )
-    (property "Footprint" "Connector_Harwin:Harwin_M20-89008xx_1x08_P2.54mm_Horizontal" (id 2) (at 124.46 139.7 0)
+    (property "Footprint" "" (id 2) (at 124.46 139.7 0)
       (effects (font (size 1.27 1.27)) hide)
     )
@@
       (effects (font (size 1.27 1.27)) (justify right))
     )
-    (property "Footprint" "Connector_Harwin:Harwin_M20-89008xx_1x08_P2.54mm_Horizontal" (id 2) (at 283.21 39.37 0)
+    (property "Footprint" "" (id 2) (at 283.21 39.37 0)
       (effects (font (size 1.27 1.27)) hide)
     )
@@
       (effects (font (size 1.27 1.27)) (justify right))
     )
-    (property "Footprint" "Connector_Harwin:Harwin_M20-89008xx_1x08_P2.54mm_Horizontal" (id 2) (at 283.21 26.67 0)
-      (effects (font (size 1.27 1.27)) hide)
-    )
+    (property "Footprint" "" (id 2) (at 283.21 26.67 0)
+      (effects (font (size 1.27 1.27)) hide)
+    )
